File: hardware/OSCAR.sch (KiCad schematic (older format))
At the start: 47 parts

Commit message: Updated PDF and labels
Other:
- note added: "+- 18V Regulator"
Changed lines of the file:
@@
 Wire Wire Line
 	4100 10450 4350 10450
+Text Notes 3750 9450 2    60   ~ 0
++- 18V Regulator
 $EndSCHEMATC
